File: keeb/keeb.kicad_pcb (KiCad board)
At the start: 2 copper layers, 305 x 95.4 mm, 137 parts, among them SW1 SW_Push, SW10 SW_Push, SW11 SW_Push, SW12 SW_Push, SW13 SW_Push, SW14 SW_Push, SW15 SW_Push, SW16 SW_Push, SW17 SW_Push, SW18 SW_Push, SW19 SW_Push, SW2 SW_Push, SW20 SW_Push, SW21 SW_Push, SW22 SW_Push, SW23 SW_Push, SW24 SW_Push, SW25 SW_Push, SW26 SW_Push, SW27 SW_Push, SW28 SW_Push, SW29 SW_Push, SW3 SW_Push, SW30 SW_Push, SW31 SW_Push, SW32 SW_Push, SW33 SW_Push, SW34 SW_Push, SW35 SW_Push, SW36 SW_Push, SW37 SW_Push, SW38 SW_Push, SW39 SW_Push, SW4 SW_Push, SW40 SW_Push, SW41 SW_Push, SW42 SW_Push, SW43 SW_Push, SW44 SW_Push, SW45 SW_Push, SW46 SW_Push, SW47 SW_Push, SW48 SW_Push, SW49 SW_Push, SW5 SW_Push, SW50 SW_Push, SW51 SW_Push, SW52 SW_Push, SW53 SW_Push, SW54 SW_Push, SW55 SW_Push, SW56 SW_Push, SW57 SW_Push, SW58 SW_Push, SW59 SW_Push, SW6 SW_Push, SW60 SW_Push, SW61 SW_Push, SW62 SW_Push, SW63 SW_Push, SW64 SW_Push, SW65 SW_Push, SW66 SW_Push, SW67 SW_Push, SW68 SW_Push, SW7 SW_Push, SW8 SW_Push, SW9 SW_Push

Commit message: submission
Parts:
- added G***: LOGO, highway:qr1, F.Cu at (137.8, 158.6)
- added G***: LOGO, highway:sbkeeb, F.Cu at (102.2, 61.6)
- added G***: LOGO, highway:hc, F.Cu at (186.8, 58.1)
- added G***: LOGO, highway:SBfinal, F.Cu at (259.1, 59.9)
- added G***: LOGO, highway:qr2, F.Cu at (206.0, 158.6)
- added SW69: RotaryEncoder_Switch_MP, ScottoKeebs_Scotto:Encoder_EC11_MX, F.Cu at (68.8, 63.0)
- added SW70: RotaryEncoder_Switch_MP, ScottoKeebs_Scotto:Encoder_EC11_MX, F.Cu at (49.7, 63.0)
- SW1, SW10, SW11, SW12, SW13, SW14, SW15, SW16, SW17, SW18, SW19, SW2, SW20, SW21, SW22, SW23, SW24, SW25, SW26, SW27, SW28, SW29, SW3, SW30, SW31, SW32, SW33, SW34, SW35, SW36, SW37, SW38, SW39, SW4, SW40, SW41, SW42, SW43, SW44, SW45, SW46, SW47, SW48, SW49, SW5, SW50, SW51, SW52, SW53, SW54, SW55, SW56, SW57, SW58, SW59, SW6, SW60, SW61, SW62, SW63, SW64, SW65, SW66, SW67, SW68, SW7, SW8, SW9: footprint Button_Switch_Keyboard:SW_Cherry_MX_1.00u_PCB -> Button_Switch_Keyboard:SW_Cherry_MX_1.00u_PCB_Sharon
- moved A1 128.6 mm to (294.2, 68.1)
- moved D13 34.4 mm to (287.8, 86.0)
- moved D19 34.4 mm to (125.9, 105.1)
- moved D21 34.4 mm to (164.0, 105.1)
- moved D24 34.4 mm to (221.2, 105.1)
- moved D35 34.4 mm to (149.7, 124.1)
- moved D37 34.4 mm to (187.8, 124.1)
- moved D40 34.4 mm to (245.0, 124.1)
- moved D41 34.4 mm to (264.0, 124.1)
- moved D48 34.4 mm to (140.2, 143.2)
- moved D51 34.4 mm to (197.3, 143.2)
- moved D53 34.4 mm to (235.4, 143.2)
- moved D56 34.4 mm to (299.7, 143.2)
- moved D7 34.4 mm to (173.5, 86.0)
- moved D9 34.4 mm to (211.6, 86.0)
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Connections:
- net Net-(A1-GND-Pad13) renamed GND
- A1 pad 1: unconnected-(A1-GPIO0-Pad1) -> Net-(A1-GPIO0)
- A1 pad 2: unconnected-(A1-GPIO1-Pad2) -> Net-(A1-GPIO1)
- A1 pad 29: unconnected-(A1-GPIO22-Pad29) -> Net-(A1-GPIO22)
- A1 pad 31: unconnected-(A1-GPIO26_ADC0-Pad31) -> Net-(A1-GPIO26_ADC0)
- A1 pad 32: unconnected-(A1-GPIO27_ADC1-Pad32) -> Net-(A1-GPIO27_ADC1)
- A1 pad 34: unconnected-(A1-GPIO28_ADC2-Pad34) -> Net-(A1-GPIO28_ADC2)
Routing:
- net r5: track 0.00 -> 420.6 mm
- net r4: track 10.2 -> 388.4 mm
- net r3: track 17.7 -> 370.6 mm
- net r2: track 0.00 -> 350.4 mm
- net C1: track 0.00 -> 338.9 mm
- net C2: track 0.00 -> 330.2 mm
- net r1: track 0.00 -> 330.0 mm
- net C3: track 0.00 -> 311.3 mm
- net Net-(A1-GPIO28_ADC2): track 0.00 -> 279.1 mm
- net Net-(A1-GPIO27_ADC1): track 0.00 -> 276.6 mm
- net C4: track 0.00 -> 270.8 mm
- net Net-(A1-GPIO26_ADC0): track 0.00 -> 267.8 mm, vias 0 -> 1
- net GND: track 0.00 -> 264.5 mm
- net C5: track 0.00 -> 256.8 mm
- net Net-(A1-GPIO22): track 0.00 -> 252.7 mm
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Other:
- board size 305 x 95.4 mm -> 309.1 x 121.7 mm
